File: PCB/PCB.kicad_sch (KiCad schematic)
At the start: 0 parts

Commit message: commit ma balls
Parts:
- added D1, D2, D3, D4, D5, D6: D_Small, Diode_THT:D_DO-35_SOD27_P7.62mm_Horizontal, symbol Device:D_Small
- added M1, M2: Motor_Servo, Connector_PinSocket_2.54mm:PinSocket_1x03_P2.54mm_Vertical, symbol Motor:Motor_Servo
- added SW1, SW2: RotaryEncoder_Switch, Rotary_Encoder:RotaryEncoder_Alps_EC11E-Switch_Vertical_H20mm, symbol Device:RotaryEncoder_Switch
- added SW3, SW4, SW5, SW6: SW_Push, Taranium-libs:SW_Cherry_MX_1.00u_PCB, symbol Switch:SW_Push
- added U1: XIAO-RP2040-DIP, Taranium-libs:XIAO-RP2040-DIP, symbol Seeed_Studio_XIAO_Series:XIAO-RP2040-DIP
Connections:
- new net: D5.2 (A), SW5.2
- new net: D1.2 (A), SW2.S1
- new net: D6.2 (A), SW6.2
- new net: D4.2 (A), SW4.2
- new net: D2.2 (A), SW1.S1
- new net: D3.2 (A), SW3.2
- new net +3V3: U1.12 (3V3)
- new net +5V: M1.2 (+), M2.2 (+), U1.14 (VBUS)
- new net A1: SW1.A, U1.6 (P7_SCL_D5)
- new net A2: SW2.A, U1.10 (P4_D9_MISO)
- new net B1: SW1.B, U1.5 (P6_SDA_D4)
- new net B2: SW2.B, U1.9 (P2_D8_SCK)
- new net C1: SW1.S2, SW4.1, U1.3 (P28_A2_D2)
- new net C2: SW3.1, SW5.1, U1.7 (P0_D6_TX)
- new net C3: SW2.S2, SW6.1, U1.8 (P1_D7_RX)
- new net GND: M1.3 (-), M2.3 (-), SW1.C, SW2.C, U1.13 (GND)
- new net R1: D1.1 (K), D2.1 (K), D3.1 (K), U1.4 (P29_A3_D3)
- new net R2: D4.1 (K), D5.1 (K), D6.1 (K), U1.2 (P27_A1_D1)
- new net S1: M1.1 (PWM), U1.1 (P26_A0_D0)
- new net S2: M2.1 (PWM), U1.11 (P3_D10_MOSI)
