File: PCB/PCB.kicad_pcb (KiCad board)
At the start: 2 copper layers, 62 x 67 mm, 16 parts, among them M1 Conn_01x02_Pin, M2 Conn_01x02_Pin, SW1 RotaryEncoder_Switch, SW2 RotaryEncoder_Switch, SW3 SW_Push, SW4 SW_Push, SW5 SW_Push, SW6 SW_Push, U1 L293D

Commit message: potato
Parts:
- moved M2 1.21 mm to (190.5, 75.3)
- moved M1 0.60 mm to (134.0, 77.9)
Routing:
- net M2 P2: track 4.78 -> 5.99 mm
- net M2 P1: track 4.70 -> 4.20 mm
Changed lines of the file:
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@@
 	(footprint "Connector_PinHeader_2.54mm:PinHeader_1x02_P2.54mm_Vertical"
 		(layer "F.Cu")
-		(at 134 77.275 180)
+		(at 134 77.875 180)
 		(descr "Through hole straight pin header, 1x02, 2.54mm pitch, single row")
 		(tags "Through hole pin header THT 1x02 2.54mm single row")
@@
 	(footprint "Connector_PinHeader_2.54mm:PinHeader_1x02_P2.54mm_Vertical"
 		(layer "F.Cu")
-		(at 190.5 74.125)
+		(at 190.5 75.335)
 		(descr "Through hole straight pin header, 1x02, 2.54mm pitch, single row")
 		(tags "Through hole pin header THT 1x02 2.54mm single row")
@@
 	(segment
 		(start 175.110314 83.316)
-		(end 140.041 83.316)
+		(end 139.441 83.316)
 		(width 0.5)
 		(layer "B.Cu")
@@
 	)
 	(segment
-		(start 140.041 83.316)
+		(start 179.195 79.231314)
+		(end 175.110314 83.316)
+		(width 0.5)
+		(layer "B.Cu")
+		(net 24)
+	)
+	(segment
+		(start 134 77.875)
 		(end 134 77.275)
 		(width 0.5)
@@
 	)
 	(segment
-		(start 179.195 79.231314)
-		(end 175.110314 83.316)
+		(start 139.441 83.316)
+		(end 134 77.875)
 		(width 0.5)
 		(layer "B.Cu")
@@
 	)
 	(segment
-		(start 175.105 67.4)
-		(end 141.335 67.4)
+		(start 141.935 67.4)
+		(end 134 75.335)
 		(width 0.5)
 		(layer "B.Cu")
@@
 	)
 	(segment
-		(start 141.335 67.4)
-		(end 134 74.735)
+		(start 175.105 67.4)
+		(end 141.935 67.4)
 		(width 0.5)
 		(layer "B.Cu")
@@
 	)
 	(segment
-		(start 187.865 71.49)
+		(start 190.5 75.335)
 		(end 190.5 74.125)
 		(width 0.5)
@@
 	)
 	(segment
-		(start 188.055 79.11)
-		(end 190.5 76.665)
+		(start 190.5 74.125)
+		(end 187.865 71.49)
+		(width 0.5)
+		(layer "F.Cu")
+		(net 26)
+	)
+	(segment
+		(start 189.265 79.11)
+		(end 186.815 79.11)
 		(width 0.5)
 		(layer "F.Cu")
@@
 	)
 	(segment
-		(start 186.815 79.11)
-		(end 188.055 79.11)
+		(start 190.5 77.875)
+		(end 189.265 79.11)
 		(width 0.5)
 		(layer "F.Cu")

Commit message: commit
Other:
- board text added: "Potato"
- board text added: "Taran-the-Idiot"
- board text added: "taranium.dev"
Changed lines of the file:
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@@
 		)
+	)
+	(gr_poly
+		(pts
+			(xy 163.436459 95.169749) (xy 163.436459 103.58125) (xy 169.654168 89.176817) (xy 166.107825 89.176817)
+		)
+		(stroke
+			(width 0)
+			(type solid)
+		)
+		(fill yes)
+		(layer "B.SilkS")
+	)
+	(gr_poly
+		(pts
+			(xy 128.563873 59.68947) (xy 127.463873 85.18947) (xy 158.263873 59.28947) (xy 132.863873 57.68947)
+		)
+		(stroke
+			(width 0.1)
+			(type solid)
+		)
+		(fill yes)
+		(layer "B.SilkS")
+	)
+	(gr_poly
+		(pts
+			(xy 159.600001 103.448958) (xy 162.907294 103.448958) (xy 162.907294 88.5) (xy 159.600001 88.5)
+		)
+		(stroke
+			(width 0)
+			(type solid)
+		)
+		(fill yes)
+		(layer "B.SilkS")
+	)
+	(gr_rect
+		(start 188.0875 49.3)
+		(end 195.35 123.6)
+		(stroke
+			(width 0.1)
+			(type solid)
+		)
+		(fill yes)
+		(layer "B.SilkS")
+	)
+	(gr_poly
+		(pts
+			(xy 194.073313 60.708805) (xy 168.573313 59.608805) (xy 194.473313 90.408805) (xy 196.073313 65.008805)
+		)
+		(stroke
+			(width 0.1)
+			(type solid)
+		)
+		(fill yes)
+		(layer "B.SilkS")
+	)
+	(gr_poly
+		(pts
+			(xy 152.853125 103.406491) (xy 155.880225 103.406491) (xy 155.880225 89.097905) (xy 152.853125 89.097905)
+		)
+		(stroke
+			(width 0)
+			(type solid)
+		)
+		(fill yes)
+		(layer "B.SilkS")
+	)
+	(gr_poly
+		(pts
+			(xy 159.070835 103.448958) (xy 159.070835 95.492407) (xy 156.304087 89.029166) (xy 152.870325 89.029166)
+		)
+		(stroke
+			(width 0)
+			(type solid)
+		)
+		(fill yes)
+		(layer "B.SilkS")
+	)
+	(gr_poly
+		(pts
+			(xy 148.487502 84.135049) (xy 151.794794 104.110415) (xy 151.794794 82.811458)
+		)
+		(stroke
+			(width 0)
+			(type solid)
+		)
+		(fill yes)
+		(layer "B.SilkS")
+	)
+	(gr_poly
+		(pts
+			(xy 193.9 129.4) (xy 195 103.9) (xy 164.2 129.8) (xy 189.6 131.4)
+		)
+		(stroke
+			(width 0.1)
+			(type solid)
+		)
+		(fill yes)
+		(layer "B.SilkS")
+	)
+	(gr_poly
+		(pts
+			(xy 152.853125 88.5) (xy 169.654168 88.5) (xy 169.654168 84.266667) (xy 152.853125 84.266667)
+		)
+		(stroke
+			(width 0)
+			(type solid)
+		)
+		(fill yes)
+		(layer "B.SilkS")
+	)
+	(gr_poly
+		(pts
+			(xy 152.853125 82.540591) (xy 152.853125 83.472917) (xy 169.654168 83.472917) (xy 169.654168 82.540591)
+			(xy 161.253647 80.694792)
+		)
+		(stroke
+			(width 0)
+			(type solid)
+		)
+		(fill yes)
+		(layer "B.SilkS")
+	)
+	(gr_rect
+		(start 124.1 58.4)
+		(end 198.4 65.6625)
+		(stroke
+			(width 0.1)
+			(type solid)
+		)
+		(fill yes)
+		(layer "B.SilkS")
+	)
+	(gr_poly
+		(pts
+			(xy 166.593468 103.454779) (xy 169.629033 103.454779) (xy 169.629033 89.161458) (xy 166.593468 89.161458)
+		)
+		(stroke
+			(width 0)
+			(type solid)
+		)
+		(fill yes)
+		(layer "B.SilkS")
+	)
+	(gr_rect
+		(start 124.85 124)
+		(end 199.15 131.2625)
+		(stroke
+			(width 0.1)
+			(type solid)
+		)
+		(fill yes)
+		(layer "B.SilkS")
+	)
+	(gr_rect
+		(start 126.6875 52.9)
+		(end 133.95 127.2)
+		(stroke
+			(width 0.1)
+			(type solid)
+		)
+		(fill yes)
+		(layer "B.SilkS")
+	)
+	(gr_poly
+		(pts
+			(xy 170.712501 104.110415) (xy 174.019792 84.135049) (xy 170.712501 82.811458)
+		)
+		(stroke
+			(width 0)
+			(type solid)
+		)
+		(fill yes)
+		(layer "B.SilkS")
+	)
+	(gr_poly
+		(pts
+			(xy 161.253647 107.417706) (xy 169.788973 104.540364) (xy 152.718321 104.540364)
+		)
+		(stroke
+			(width 0)
+			(type solid)
+		)
+		(fill yes)
+		(layer "B.SilkS")
+	)
+	(gr_poly
+		(pts
+			(xy 130.7 130) (xy 156.2 131.1) (xy 130.3 100.3) (xy 128.7 125.7)
+		)
+		(stroke
+			(width 0.1)
+			(type solid)
+		)
+		(fill yes)
+		(layer "B.SilkS")
 	)
 	(gr_line
@@
 		)
 		(layer "Edge.Cuts")
+	)
+	(gr_text "Potato"
+		(at 136.3 127.1 0)
+		(layer "F.SilkS")
+		(effects
+			(font
+				(size 1 1)
+				(thickness 0.1)
+			)
+			(justify left bottom)
+		)
+	)
+	(gr_text "taranium.dev"
+		(at 138.4 69.5 0)
+		(layer "F.SilkS")
+		(effects
+			(font
+				(size 2.5 2.5)
+				(thickness 0.6)
+				(bold yes)
+			)
+			(justify left bottom)
+		)
+	)
+	(gr_text "Taran-the-Idiot"
+		(at 138.2 73.9 0)
+		(layer "F.SilkS")
+		(effects
+			(font
+				(size 2.5 2.5)
+				(thickness 0.6)
+				(bold yes)
+			)
+			(justify left bottom)
+		)
 	)
 	(segment
@@
 		)
 	)
+	(group ""
+		(members "270b924d-eb38-4b0a-bd70-eccecb5aeb20" "3394eb2c-9ffd-4a7f-b41c-8f0042c6309b"
+			"66a14c7b-d10b-4b5e-997a-bdd5a65f334e" "6acc926b-8bcc-4747-bceb-64746d85234c"
+			"86bc0bb8-7f74-4b9b-b66e-4ed078e1d718" "8ca53d12-c9a3-4cec-a971-ab416481c8fa"
+			"9695b8e7-53ca-4a54-bc5a-a703b31bf663" "b8a4f3ef-8be1-4c5b-bf40-4ecda3179620"
+			"f2d2f78e-f932-480f-b425-9d46733a7510" "f952c580-244f-455a-bd7c-0080499d8f37"
+		)
+	)
